File: testcases/test_peripherals.kicad_sch (KiCad schematic)
At the start: 2 parts, among them U1 STM32F103C8Tx, Y1 Crystal

Commit message: fixed heuristic analysis + other random things i dont rmb...
Parts:
- removed U1: STM32F103C8Tx, Package_QFP:LQFP-48_7x7mm_P0.5mm, symbol MCU_ST_STM32F1:STM32F103C8Tx
- removed Y1: Crystal, symbol Device:Crystal
- added C1: C, symbol Device:C
- added D1: LED, symbol Device:LED
- added R1: 1k, symbol Device:R
- added U1: SENSOR, symbol Custom:Sensor_I2C
Connections:
- net GND: now also C1.2, D1.1 (K), U1.2 (GND)
- new net: C1.1, R1.1
- new net: D1.2 (A), R1.2
- new net +3V3: U1.1 (VCC)
